Commit message: moveit2 wip

File: interbotix_ros_xsarms/interbotix_xsarm_descriptions/urdf/rx200.urdf.xacro (robot description, xacro)
@@ -52,13 +52,4 @@
     <dynamics friction="0.1"/>
   </joint>
-  <transmission name="trans_waist">
-    <type>transmission_interface/SimpleTransmission</type>
-    <joint name="waist">
-      <hardwareInterface>hardware_interface/EffortJointInterface</hardwareInterface>
-    </joint>
-    <actuator name="waist_motor">
-      <mechanicalReduction>1</mechanicalReduction>
-    </actuator>
-  </transmission>
   <link name="$(arg robot_name)/shoulder_link">
     <visual>
@@ -89,13 +80,4 @@
     <dynamics friction="0.1"/>
   </joint>
-  <transmission name="trans_shoulder">
-    <type>transmission_interface/SimpleTransmission</type>
-    <joint name="shoulder">
-      <hardwareInterface>hardware_interface/EffortJointInterface</hardwareInterface>
-    </joint>
-    <actuator name="shoulder_motor">
-      <mechanicalReduction>1</mechanicalReduction>
-    </actuator>
-  </transmission>
   <link name="$(arg robot_name)/upper_arm_link">
     <visual>
@@ -126,13 +108,4 @@
     <dynamics friction="0.1"/>
   </joint>
-  <transmission name="trans_elbow">
-    <type>transmission_interface/SimpleTransmission</type>
-    <joint name="elbow">
-      <hardwareInterface>hardware_interface/EffortJointInterface</hardwareInterface>
-    </joint>
-    <actuator name="elbow_motor">
-      <mechanicalReduction>1</mechanicalReduction>
-    </actuator>
-  </transmission>
   <link name="$(arg robot_name)/forearm_link">
     <visual>
@@ -163,13 +136,4 @@
     <dynamics friction="0.1"/>
   </joint>
-  <transmission name="trans_wrist_angle">
-    <type>transmission_interface/SimpleTransmission</type>
-    <joint name="wrist_angle">
-      <hardwareInterface>hardware_interface/EffortJointInterface</hardwareInterface>
-    </joint>
-    <actuator name="wrist_angle_motor">
-      <mechanicalReduction>1</mechanicalReduction>
-    </actuator>
-  </transmission>
   <link name="$(arg robot_name)/wrist_link">
     <visual>
@@ -200,13 +164,4 @@
     <dynamics friction="0.1"/>
   </joint>
-  <transmission name="trans_wrist_rotate">
-    <type>transmission_interface/SimpleTransmission</type>
-    <joint name="wrist_rotate">
-      <hardwareInterface>hardware_interface/EffortJointInterface</hardwareInterface>
-    </joint>
-    <actuator name="wrist_rotate_motor">
-      <mechanicalReduction>1</mechanicalReduction>
-    </actuator>
-  </transmission>
   <link name="$(arg robot_name)/gripper_link">
     <visual>
@@ -249,13 +204,4 @@
     <dynamics friction="0.1"/>
   </joint>
-  <transmission name="trans_gripper">
-    <type>transmission_interface/SimpleTransmission</type>
-    <joint name="gripper">
-      <hardwareInterface>hardware_interface/EffortJointInterface</hardwareInterface>
-    </joint>
-    <actuator name="gripper_motor">
-      <mechanicalReduction>1</mechanicalReduction>
-    </actuator>
-  </transmission>
   <link name="$(arg robot_name)/gripper_prop_link">
     <visual>
@@ -357,13 +303,4 @@
         <dynamics friction="0.1"/>
       </joint>
-      <transmission name="trans_left_finger">
-        <type>transmission_interface/SimpleTransmission</type>
-        <joint name="left_finger">
-          <hardwareInterface>hardware_interface/EffortJointInterface</hardwareInterface>
-        </joint>
-        <actuator name="left_finger_motor">
-          <mechanicalReduction>1</mechanicalReduction>
-        </actuator>
-      </transmission>
       <link name="$(arg robot_name)/left_finger_link">
         <visual>
@@ -397,13 +334,4 @@
         </xacro:unless>
       </joint>
-      <transmission name="trans_right_finger">
-        <type>transmission_interface/SimpleTransmission</type>
-        <joint name="right_finger">
-          <hardwareInterface>hardware_interface/EffortJointInterface</hardwareInterface>
-        </joint>
-        <actuator name="right_finger_motor">
-          <mechanicalReduction>1</mechanicalReduction>
-        </actuator>
-      </transmission>
       <link name="$(arg robot_name)/right_finger_link">
         <visual>
@@ -443,3 +371,50 @@
     <xacro:include filename="${urdf_loc}"/>
   </xacro:if>
+  <ros2_control name="XSHardwareInterface" type="system">
+    <hardware>
+      <plugin>interbotix_xs_ros_control/XSHardwareInterface</plugin>
+    </hardware>
+    <joint name="waist">
+      <command_interface name="position">
+        <param name="min">"${-pi + pi_offset}"</param>
+        <param name="max">"${pi - pi_offset}"</param>
+      </command_interface>
+      <state_interface name="position"/>
+    </joint>
+    <joint name="shoulder">
+      <command_interface name="position">
+        <param name="min">"${radians(-108)}"</param>
+        <param name="max">"${radians(113)}"</param>
+      </command_interface>
+      <state_interface name="position"/>
+    </joint>
+    <joint name="elbow">
+      <command_interface name="position">
+        <param name="min">"${radians(-108)}"</param>
+        <param name="max">"${radians(93)}"</param>
+      </command_interface>
+      <state_interface name="position"/>
+    </joint>
+    <joint name="wrist_angle">
+      <command_interface name="position">
+        <param name="min">"${radians(-100)}"</param>
+        <param name="max">"${radians(123)}"</param>
+      </command_interface>
+      <state_interface name="position"/>
+    </joint>
+    <joint name="wrist_rotate">
+      <command_interface name="position">
+        <param name="min">"${-pi + pi_offset}"</param>
+        <param name="max">"${pi - pi_offset}"</param>
+      </command_interface>
+      <state_interface name="position"/>
+    </joint>
+    <joint name="left_finger">
+      <command_interface name="position">
+        <param name="min">0.015</param>
+        <param name="max">-0.015</param>
+      </command_interface>
+      <state_interface name="position"/>
+    </joint>
+  </ros2_control>
 </robot>

File: interbotix_ros_xsarms/interbotix_xsarm_moveit/config/srdf/rx200.srdf.xacro (robot description, xacro)
@@ -30,5 +30,4 @@
         <link name="$(arg robot_name)/right_finger_link" />
     </group>
-    <!--GROUP STATES: Purpose: Define a named state for a particular group, in terms of joint values. This is useful to define states like 'folded arms'-->
     <group_state name="Home" group="interbotix_arm">
         <joint name="elbow" value="0" />
@@ -64,7 +63,5 @@
         <joint name="right_finger" value="-0.0195" />
     </group_state>
-    <!--END EFFECTOR: Purpose: Represent information about an end effector.-->
     <end_effector name="interbotix_gripper" parent_link="$(arg robot_name)/ee_gripper_link" group="interbotix_gripper" />
-    <!--DISABLE COLLISIONS: By default it is assumed that any link of the robot could potentially come into collision with any other link in the robot. This tag disables collision checking between a specified pair of links. -->
     <disable_collisions link1="$(arg robot_name)/$(arg base_link_frame)" link2="$(arg robot_name)/shoulder_link" reason="Adjacent" />
     <disable_collisions link1="$(arg robot_name)/forearm_link" link2="$(arg robot_name)/gripper_bar_link" reason="Never" />
